File: Breadboard 400/Breadboard 400.kicad_pcb (KiCad board)
At the start: 2 copper layers, 81.3 x 53.3 mm, 46 parts

Commit message: Fixed problems with the first one
Parts:
- removed the REF** at (160.0, 94.6)
- removed the REF** at (86.4, 94.6)
- moved REF** 0.90 mm to (83.8, 95.2), turned to 270 degrees
- moved REF** 0.90 mm to (162.6, 95.2), turned to 90 degrees
Routing:
- net (no net): track 1114.2 -> 1001.7 mm, vias 4 -> 0
Other:
- board text added: "BREADBOARD 400"
- board text added: "Link +"
- board text added: "Link -"
- board text added: "Revision B github.com/tebl"

Commit message: Gerber export
Parts:
- removed REF** (x2): bridge, breadboard:bridge
- removed REF** (x10): power, breadboard:power
- removed REF** (x30): section, breadboard:section
- removed REF** (x2): 1pin, mounting:M2
- added A1: PWR, breadboard:power, F.Cu at (118.1, 73.7)
- added A10: BB, breadboard:section, F.Cu at (139.7, 109.2)
- added A11: PWR, breadboard:power, F.Cu at (148.6, 119.4)
- added A12: PWR, breadboard:power, F.Cu at (87.6, 119.4)
- added A13: PWR, breadboard:power, F.Cu at (102.9, 119.4)
- added A14: PWR, breadboard:power, F.Cu at (133.3, 119.4)
- added A15: PWR, breadboard:power, F.Cu at (118.1, 119.4)
- added A16: BB, breadboard:section, F.Cu at (137.2, 109.2)
- added A17: BB, breadboard:section, F.Cu at (134.6, 109.2)
- added A18: BB, breadboard:section, F.Cu at (132.1, 109.2)
- added A19: BB, breadboard:section, F.Cu at (129.5, 109.2)
- added A2: PWR, breadboard:power, F.Cu at (148.6, 73.7)
- added A20: BB, breadboard:section, F.Cu at (127.0, 109.2)
- added A21: BB, breadboard:section, F.Cu at (88.9, 109.2)
- added A22: BB, breadboard:section, F.Cu at (116.8, 109.2)
- added A23: BB, breadboard:section, F.Cu at (119.4, 109.2)
- added A24: BB, breadboard:section, F.Cu at (86.4, 109.2)
- added A25: BB, breadboard:section, F.Cu at (111.8, 109.2)
- added A26: BB, breadboard:section, F.Cu at (109.2, 109.2)
- added A27: BB, breadboard:section, F.Cu at (106.7, 109.2)
- added A28: BB, breadboard:section, F.Cu at (104.1, 109.2)
- added A29: BB, breadboard:section, F.Cu at (101.6, 109.2)
- added A3: PWR, breadboard:power, F.Cu at (102.9, 73.7)
- added A30: BB, breadboard:section, F.Cu at (99.1, 109.2)
- added A31: BB, breadboard:section, F.Cu at (96.5, 109.2)
- added A32: BB, breadboard:section, F.Cu at (94.0, 109.2)
- added A33: BB, breadboard:section, F.Cu at (91.4, 109.2)
- added A34: BB, breadboard:section, F.Cu at (124.5, 109.2)
- added A35: BB, breadboard:section, F.Cu at (121.9, 109.2)
- added A36: BB, breadboard:section, F.Cu at (114.3, 109.2)
- added A37: BB, breadboard:section, F.Cu at (152.4, 109.2)
- added A38: BB, breadboard:section, F.Cu at (154.9, 109.2)
- added A39: BB, breadboard:section, F.Cu at (157.5, 109.2)
- added A4: PWR, breadboard:power, F.Cu at (133.3, 73.7)
- added A40: BB, breadboard:section, F.Cu at (160.0, 109.2)
- added A5: PWR, breadboard:power, F.Cu at (87.6, 73.7)
- added A6: BB, breadboard:section, F.Cu at (149.9, 109.2)
- added A7: BB, breadboard:section, F.Cu at (147.3, 109.2)
- added A8: BB, breadboard:section, F.Cu at (144.8, 109.2)
- added A9: BB, breadboard:section, F.Cu at (142.2, 109.2)
- added H1: MountingHole, mounting:M3, F.Cu at (156.2, 95.2)
- added H2: MountingHole, mounting:M3, F.Cu at (90.2, 95.2)
- added JP5: LINK_VCC, breadboard:bridge, B.Cu at (84.1, 94.4)
- added JP6: LINK_GND, breadboard:bridge, B.Cu at (162.3, 96.3)
Routing:
- net (no net): track 1001.7 -> 0.00 mm
- net /GND1: track 0.00 -> 98.2 mm
- net /VCC2: track 0.00 -> 98.1 mm
- net /VCC1: track 0.00 -> 95.6 mm
- net /GND2: track 0.00 -> 95.5 mm
- net Net-(A9-Pad2): track 0.00 -> 10.2 mm
- net Net-(A9-Pad1): track 0.00 -> 10.2 mm
- net Net-(A8-Pad2): track 0.00 -> 10.2 mm
- net Net-(A8-Pad1): track 0.00 -> 10.2 mm
- net Net-(A7-Pad2): track 0.00 -> 10.2 mm
- net Net-(A7-Pad1): track 0.00 -> 10.2 mm
- net Net-(A6-Pad2): track 0.00 -> 10.2 mm
- net Net-(A6-Pad1): track 0.00 -> 10.2 mm
- net Net-(A40-Pad2): track 0.00 -> 10.2 mm
- net Net-(A40-Pad1): track 0.00 -> 10.2 mm
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Other:
- rule pad_to_mask_clearance: 0.051 -> 0
- board text added: "A"
- board text added: "B"
- board text added: "C"
- board text added: "D"
- board text added: "E"
- board text added: "F"
- board text added: "G"
- board text added: "GND"
- board text added: "H"
- board text added: "I"
- board text added: "J"
- board text added: "Licensed under CERN OHL v1.2"
- board text added: "Revision C github.com/tebl"
- board text added: "VCC"
- board text removed: "Link +"
- board text removed: "Link -"
- board text removed: "Revision B github.com/tebl"
- board text removed: "a"
- board text removed: "b"
- board text removed: "c"
- board text removed: "d"
- board text removed: "e"
- board text removed: "f"
- board text removed: "g"
- board text removed: "i"
- board text removed: "j"
